File: hardware/bluepill_geyser.sch (KiCad schematic (older format))
At the start: 20 parts, among them J4 Conn_01x04, J5 Conn_01x04

Commit message: Sample analogs with timer2 interrupt every 250us for 80 samples, enabling us to calculate 20ms RMS
Parts:
- removed D?: 1N4007, Diode_THT:D_DO-41_SOD81_P10.16mm_Horizontal, symbol Diode:1N4007
- removed Q?: BC237, Package_TO_SOT_THT:TO-92_Inline, symbol Transistor_BJT:BC237
- removed R?: 100K, symbol Device:R
- removed R?: 22K, symbol Device:R
- removed R?: 47K, symbol Device:R
- removed R?: 220R, symbol Device:R
- removed R?: 100R, symbol Device:R
- added R?: 22K, symbol Device:R
- added R?: 10K, symbol Device:R
- added U? (x5): LM324, symbol Amplifier_Operational:LM324
- C?: value 47uF -> 100nF
- R?: value 10K -> 470K
- R?: value 22K -> 10K
Connections:
- net labels added: NEG_CURRENT_TRANSFORMER, POS_CURRENT_TRANSFORMER
- net labels removed: CURRENT_TRANSFORMER
- wire segments 54 -> 80
Other:
- moved on the sheet: C1, R?
